File: keyboard_68.sch (KiCad schematic (older format))
At the start: 19 parts, among them J1 Conn_01x02_Male, J70 Conn_02x03_Odd_Even, SW1 SW_Push, U1 USB_C, U2 nRF52840_som

Commit message: changed inductor and usb connector
Parts:
- U1: footprint Connector_USB:USB_C_Receptacle_Amphenol_12401610E4-2A -> USB_C_Receptacle_Amphenol_12401610E4-2A:USB_C_Receptacle_Amphenol_12401610E4-2A
Changed lines of the file:
@@
 EESchema Schematic File Version 4
+LIBS:keyboard_68-cache
 EELAYER 30 0
 EELAYER END
@@
 F 0 "U1" H 2150 3400 50  0000 C CNN
 F 1 "USB_C" H 2150 3200 50  0000 C CNN
-F 2 "Connector_USB:USB_C_Receptacle_Amphenol_12401610E4-2A" H 2150 3800 50  0001 C CNN
+F 2 "USB_C_Receptacle_Amphenol_12401610E4-2A:USB_C_Receptacle_Amphenol_12401610E4-2A" H 2150 3800 50  0001 C CNN
 F 3 "https://www.amphenol-icc.com/media/wysiwyg/files/drawing/12401610e4x2a.pdf" H 2150 3800 50  0001 C CNN
 F 4 " 12401610E4#2ACT-ND " H 2150 3200 50  0001 C CNN "DigiKey"

Commit message: changed wrong partnumber of reset switch
Parts:
- SW1: Description (none) -> SWITCH TACTILE SPST-NO 0.05A 12V; DigiKey P10851SCT-ND -> P10851SCT-ND; Digikey (none) -> P10851SCT-ND; LCSC C79174 -> C128539; MPN (none) -> EVQ-PUJ02K; Manufacturer (none) -> Panasonic Electronic Components; Spec (none) -> SPEC
Changed lines of the file:
@@
 F 2 "Button_Switch_SMD:Panasonic_EVQPUJ_EVQPUA" H 10100 5150 50  0001 C CNN
 F 3 "https://industrial.panasonic.com/cdbs/www-data/pdf/ATK0000/ATK0000C382.pdf" H 10100 5150 50  0001 C CNN
-F 4 " P10851SCT-ND " H 10100 4950 50  0001 C CNN "DigiKey"
-F 5 "C79174" H 10100 4950 50  0001 C CNN "LCSC"
+F 4 "P10851SCT-ND " H 10100 4950 50  0001 C CNN "DigiKey"
+F 5 "C128539" H 10100 4950 50  0001 C CNN "LCSC"
+F 6 "SWITCH TACTILE SPST-NO 0.05A 12V" H 10100 4950 50  0001 C CNN "Description"
+F 7 "P10851SCT-ND " H 10100 4950 50  0001 C CNN "Digikey"
+F 8 "EVQ-PUJ02K" H 10100 4950 50  0001 C CNN "MPN"
+F 9 "Panasonic Electronic Components" H 10100 4950 50  0001 C CNN "Manufacturer"
+F 10 "SPEC" H 10100 4950 50  0001 C CNN "Spec"
 	1    10100 4950
 	-1   0    0    -1

Commit message: reset switch model added
Parts:
- SW1: footprint Button_Switch_SMD:Panasonic_EVQPUJ_EVQPUA -> custom_footprints:Panasonic_EVQPUJ_EVQPUA
Changed lines of the file:
@@
 F 0 "SW1" V 10100 5250 50  0000 R CNN
 F 1 "SW_Push" V 9950 5300 50  0000 R CNN
-F 2 "Button_Switch_SMD:Panasonic_EVQPUJ_EVQPUA" H 10100 5150 50  0001 C CNN
+F 2 "custom_footprints:Panasonic_EVQPUJ_EVQPUA" H 10100 5150 50  0001 C CNN
 F 3 "https://industrial.panasonic.com/cdbs/www-data/pdf/ATK0000/ATK0000C382.pdf" H 10100 5150 50  0001 C CNN
 F 4 "P10851SCT-ND " H 10100 4950 50  0001 C CNN "DigiKey"

Commit message: changed some value fields
Parts:
- SW1: value SW_Push -> EVQPUJ02K / EVQPUA02K
Changed lines of the file:
@@
 P 10100 4950
 F 0 "SW1" V 10100 5250 50  0000 R CNN
-F 1 "SW_Push" V 9950 5300 50  0000 R CNN
+F 1 "EVQPUJ02K / EVQPUA02K" H 10400 4750 50  0001 R CNN
 F 2 "custom_footprints:Panasonic_EVQPUJ_EVQPUA" H 10100 5150 50  0001 C CNN
 F 3 "https://industrial.panasonic.com/cdbs/www-data/pdf/ATK0000/ATK0000C382.pdf" H 10100 5150 50  0001 C CNN
