File: keyboard_68.sch (KiCad schematic (older format))
At the start: 24 parts, among them J1 Conn_01x02_Male, J70 Conn_02x03_Odd_Even, J71 Conn_01x04, J72 USB_C_Receptacle_USB2.0, SW1 EVQPUJ02K / EVQPUA02K, SW2 SW_SPDT, U2 nrf52840_module, U4 SN74LVC1T45DBV

Commit message: finalize for m.2 module
Parts:
- removed J71: Conn_01x04, Connector_PinHeader_2.54mm:PinHeader_1x04_P2.54mm_Horizontal, symbol Connector_Generic:Conn_01x04
- removed U2: nrf52840_module, custom_footprints:nrf52840_module, symbol nRF52840_module:nrf52840_module
- added J71: Conn_01x06, Connector_PinHeader_2.54mm:PinHeader_1x06_P2.54mm_Horizontal, symbol Connector_Generic:Conn_01x06
- added J73: Bus_M.2_Socket_B, custom_footprints:te_connectivity_121991190, symbol bus_m.2_socket_b:Bus_M.2_Socket_B
- FB1, FB2, FB3: symbol Device:Ferrite_Bead_Small -> keyboard_68-rescue:Ferrite_Bead_Small-Device
- J72: symbol Connector:USB_C_Receptacle_USB2.0 -> keyboard_68-rescue:USB_C_Receptacle_USB2.0-Connector
Connections:
- net COLUMN_0: now also J73.53 (GPIO_11)
- net COLUMN_1: now also J73.55 (GPIO_10)
- net COLUMN_2: now also J73.43 (GPIO_3)
- net COLUMN_3: now also J73.60 (GPIO_22_LEDG)
- net COLUMN_4: now also J73.56 (GPIO_24_AIN)
- net COLUMN_5: now also J73.38 (GPIO_9)
- net COLUMN_6: now also J73.31 (GPIO_7)
- net COLUMN_7: now also J73.35 (GPIO_6_NFC1)
- net COLUMN_8: now also J73.40 (GPIO_12)
- net D+: now also J73.7 (USB_D+)
- net D-: now also J73.9 (USB_D-)
- net GND: now also J73.11 (GND), J73.27 (GND), J73.3 (GND), J73.33 (GND), J73.39 (GND), J73.45 (GND), J73.5 (GND), J73.51 (GND), J73.57 (GND), J73.71 (GND), J73.73 (GND)
- net GPIO_0: now also J71.3 (Pin_3), J73.46 (GPIO_15)
- net GPIO_1: now also J71.4 (Pin_4), J73.48 (GPIO_16)
- net GPIO_2: now also J71.5 (Pin_5), J73.50 (GPIO_0_AIN)
- net GPIO_3: now also J71.6 (Pin_6), J73.52 (GPIO_1)
- net LLS_INPUT: now also J73.32 (GPIO_8_SWO)
- net ROW_0: now also J73.22 (GPIO_17)
- net ROW_1: now also J73.44 (GPIO_14)
- net ROW_2: now also J73.24 (GPIO_18)
- net ROW_3: now also J73.42 (GPIO_13)
- net ROW_4: now also J73.37 (GPIO_5_NFC2)
- net ROW_5: now also J73.41 (GPIO_4)
- net ROW_6: now also J73.62 (GPIO_21_LEDR)
- net ROW_7: now also J73.58 (GPIO_23_AIN_LEDB)
- net SWCLK: now also J73.36 (SWDCLK)
- net SWDIO: now also J73.34 (SWDIO)
- net VBUS: now also J73.21 (VBUS)
- net VDD_BAT: now also J73.66 (VDD_BAT)
- net VDD_nRF: now also J73.2 (3.3V), J73.4 (3.3V), J73.70 (3.3V), J73.72 (3.3V), J73.74 (3.3V)
- net VDIV: now also J73.54 (GPIO_2_AIN)
- net nRST: now also J73.30 (P1.18_RESET)
- new net GPIO_4: J71.2 (Pin_2), J73.28 (GPIO_19)
- new net GPIO_5: J71.1 (Pin_1), J73.26 (GPIO_20)
Other:
- moved on the sheet: C2, R5, SW1
