File: power.sch (KiCad schematic (older format))
At the start: 13 parts, among them Q1 DMG2305, U3 MT3608

Commit message: changed inductor and usb connector
Parts:
- L1: footprint Inductor_SMD:L_7.3x7.3_H4.5 -> L_3x3_H1.5:L_3x3_H1.5; Description (none) -> Power Inductors 22uH ±20% 650mA SMD,3x3x1.5mm; LCSC C27442 -> C285838; MPN (none) -> LVS303015-220M-N; Manufacturer (none) -> Chilisin Elec; Spec (none) -> SPEC
Changed lines of the file:
@@
 EESchema Schematic File Version 4
+LIBS:keyboard_68-cache
 EELAYER 30 0
 EELAYER END
@@
 F 0 "L1" V 2385 900 50  0000 C CNN
 F 1 "22µH" V 2294 900 50  0000 C CNN
-F 2 "Inductor_SMD:L_7.3x7.3_H4.5" H 2200 900 50  0001 C CNN
-F 3 "~" H 2200 900 50  0001 C CNN
-F 4 "C27442" H 2200 900 50  0001 C CNN "LCSC"
+F 2 "L_3x3_H1.5:L_3x3_H1.5" H 2200 900 50  0001 C CNN
+F 3 "https://datasheet.lcsc.com/szlcsc/Chilisin-Elec-LVS303015-220M-N_C285838.pdf" H 2200 900 50  0001 C CNN
+F 4 "C285838" H 2200 900 50  0001 C CNN "LCSC"
+F 5 "Power Inductors 22uH ±20% 650mA SMD,3x3x1.5mm" H 2200 900 50  0001 C CNN "Description"
+F 6 "LVS303015-220M-N" H 2200 900 50  0001 C CNN "MPN"
+F 7 "Chilisin Elec" H 2200 900 50  0001 C CNN "Manufacturer"
+F 8 "SPEC" H 2200 900 50  0001 C CNN "Spec"
 	1    2200 900
 	0    -1   -1   0

Commit message: changed some value fields
Parts:
- C73, C74: value 22µF -> 22uF
- L1: value 22µH -> 22uH
Changed lines of the file:
@@
 AR Path="/6178D778/61846306" Ref="L1"  Part="1"
 F 0 "L1" V 2385 900 50  0000 C CNN
-F 1 "22µH" V 2294 900 50  0000 C CNN
+F 1 "22uH" V 2294 900 50  0000 C CNN
 F 2 "L_3x3_H1.5:L_3x3_H1.5" H 2200 900 50  0001 C CNN
 F 3 "https://datasheet.lcsc.com/szlcsc/Chilisin-Elec-LVS303015-220M-N_C285838.pdf" H 2200 900 50  0001 C CNN
@@
 AR Path="/6178D778/61846319" Ref="C74"  Part="1"
 F 0 "C74" H 3592 1246 50  0000 L CNN
-F 1 "22µF" H 3592 1155 50  0000 L CNN
+F 1 "22uF" H 3592 1155 50  0000 L CNN
 F 2 "Capacitor_SMD:C_0805_2012Metric" H 3500 1200 50  0001 C CNN
 F 3 "https://datasheet.lcsc.com/szlcsc/Murata-Electronics-GRM21BR61E226ME44L_C86816.pdf" H 3500 1200 50  0001 C CNN
@@
 AR Path="/6178D778/6184631F" Ref="C73"  Part="1"
 F 0 "C73" H 1308 1154 50  0000 R CNN
-F 1 "22µF" H 1308 1245 50  0000 R CNN
+F 1 "22uF" H 1308 1245 50  0000 R CNN
 F 2 "Capacitor_SMD:C_0805_2012Metric" H 1400 1200 50  0001 C CNN
 F 3 "https://datasheet.lcsc.com/szlcsc/Murata-Electronics-GRM21BR61E226ME44L_C86816.pdf" H 1400 1200 50  0001 C CNN
