File: power.sch (KiCad schematic (older format))
At the start: 13 parts, among them Q1 DMG2305, U3 MT3608

Commit message: add lls, switch and spare gpio connector
Parts:
- U3: Spec (none) -> SPEC
Changed lines of the file:
@@
 F 3 "https://datasheet.lcsc.com/szlcsc/XI-AN-Aerosemi-Tech-MT3608_C84817.pdf" H 2150 1500 60  0001 C CNN
 F 4 "C84817" H 2150 1500 50  0001 C CNN "LCSC"
+F 5 "SPEC" H 2150 1500 50  0001 C CNN "Spec"
 	1    2150 1500
 	1    0    0    -1
