File: keyboard_68.kicad_pcb (KiCad board)
At the start: 2 copper layers, 330 x 106 mm, 308 parts, among them J1 Conn_01x02_Male, J10 Conn_01x02_Female, J11 Conn_01x02_Female, J12 Conn_01x02_Female, J13 Conn_01x02_Female, J14 Conn_01x02_Female, J15 Conn_01x02_Female, J16 Conn_01x02_Female, J17 Conn_01x02_Female, J18 Conn_01x02_Female, J19 Conn_01x02_Female, J2 Conn_01x02_Female, J20 Conn_01x02_Female, J21 Conn_01x02_Female, J22 Conn_01x02_Female, J23 Conn_01x02_Female, J24 Conn_01x02_Female, J25 Conn_01x02_Female, J26 Conn_01x02_Female, J27 Conn_01x02_Female, J28 Conn_01x02_Female, J29 Conn_01x02_Female, J3 Conn_01x02_Female, J30 Conn_01x02_Female, J31 Conn_01x02_Female, J32 Conn_01x02_Female, J33 Conn_01x02_Female, J34 Conn_01x02_Female, J35 Conn_01x02_Female, J36 Conn_01x02_Female, J37 Conn_01x02_Female, J38 Conn_01x02_Female, J39 Conn_01x02_Female, J4 Conn_01x02_Female, J40 Conn_01x02_Female, J41 Conn_01x02_Female, J42 Conn_01x02_Female, J43 Conn_01x02_Female, J44 Conn_01x02_Female, J45 Conn_01x02_Female, J46 Conn_01x02_Female, J47 Conn_01x02_Female, J48 Conn_01x02_Female, J49 Conn_01x02_Female, J5 Conn_01x02_Female, J50 Conn_01x02_Female, J51 Conn_01x02_Female, J52 Conn_01x02_Female, J53 Conn_01x02_Female, J54 Conn_01x02_Female, J55 Conn_01x02_Female, J56 Conn_01x02_Female, J57 Conn_01x02_Female, J58 Conn_01x02_Female, J59 Conn_01x02_Female, J6 Conn_01x02_Female, J60 Conn_01x02_Female, J61 Conn_01x02_Female, J62 Conn_01x02_Female, J63 Conn_01x02_Female, J64 Conn_01x02_Female, J65 Conn_01x02_Female, J66 Conn_01x02_Female, J67 Conn_01x02_Female, J68 Conn_01x02_Female, J69 Conn_01x02_Female, J7 Conn_01x02_Female, J70 Conn_02x03_Odd_Even, J8 Conn_01x02_Female, J9 Conn_01x02_Female, Q1 DMG2305, SW1 EVQPUJ02K / EVQPUA02K, U1 USB_C, U2 nrf52840_module, U3 MT3608

Commit message: page title etc
Parts:
- moved C12 38.4 mm to (145.1, 186.0)
- moved C14 38.4 mm to (240.4, 186.0)
- moved C2 38.4 mm to (365.9, 217.5)
- moved C20 38.4 mm to (259.3, 186.0)
- moved C22 38.4 mm to (88.4, 186.0)
- moved C23 38.4 mm to (297.9, 186.0)
- moved C26 38.4 mm to (126.0, 186.0)
- moved C30 38.4 mm to (322.3, 186.0)
- moved C32 38.4 mm to (221.3, 186.0)
- moved C38 38.4 mm to (107.0, 186.0)
- moved C42 38.4 mm to (183.2, 186.0)
- moved C48 38.4 mm to (202.6, 186.0)
- moved C5 38.4 mm to (164.4, 186.0)
- moved C52 38.4 mm to (65.0, 186.0)
- moved C73 38.4 mm to (314.0, 209.3)
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