File: keyboard_68.kicad_pcb (KiCad board)
At the start: 2 copper layers, 330 x 106 mm, 308 parts, among them J1 Conn_01x02_Male, J10 Conn_01x02_Female, J11 Conn_01x02_Female, J12 Conn_01x02_Female, J13 Conn_01x02_Female, J14 Conn_01x02_Female, J15 Conn_01x02_Female, J16 Conn_01x02_Female, J17 Conn_01x02_Female, J18 Conn_01x02_Female, J19 Conn_01x02_Female, J2 Conn_01x02_Female, J20 Conn_01x02_Female, J21 Conn_01x02_Female, J22 Conn_01x02_Female, J23 Conn_01x02_Female, J24 Conn_01x02_Female, J25 Conn_01x02_Female, J26 Conn_01x02_Female, J27 Conn_01x02_Female, J28 Conn_01x02_Female, J29 Conn_01x02_Female, J3 Conn_01x02_Female, J30 Conn_01x02_Female, J31 Conn_01x02_Female, J32 Conn_01x02_Female, J33 Conn_01x02_Female, J34 Conn_01x02_Female, J35 Conn_01x02_Female, J36 Conn_01x02_Female, J37 Conn_01x02_Female, J38 Conn_01x02_Female, J39 Conn_01x02_Female, J4 Conn_01x02_Female, J40 Conn_01x02_Female, J41 Conn_01x02_Female, J42 Conn_01x02_Female, J43 Conn_01x02_Female, J44 Conn_01x02_Female, J45 Conn_01x02_Female, J46 Conn_01x02_Female, J47 Conn_01x02_Female, J48 Conn_01x02_Female, J49 Conn_01x02_Female, J5 Conn_01x02_Female, J50 Conn_01x02_Female, J51 Conn_01x02_Female, J52 Conn_01x02_Female, J53 Conn_01x02_Female, J54 Conn_01x02_Female, J55 Conn_01x02_Female, J56 Conn_01x02_Female, J57 Conn_01x02_Female, J58 Conn_01x02_Female, J59 Conn_01x02_Female, J6 Conn_01x02_Female, J60 Conn_01x02_Female, J61 Conn_01x02_Female, J62 Conn_01x02_Female, J63 Conn_01x02_Female, J64 Conn_01x02_Female, J65 Conn_01x02_Female, J66 Conn_01x02_Female, J67 Conn_01x02_Female, J68 Conn_01x02_Female, J69 Conn_01x02_Female, J7 Conn_01x02_Female, J70 Conn_02x03_Odd_Even, J8 Conn_01x02_Female, J9 Conn_01x02_Female, Q1 DMG2305, SW1 SW_Push, U1 USB_C, U2 nRF52840_som, U3 MT3608

Commit message: added dimensions, rotate battery conn
Parts:
- moved C10 89.4 mm to (69.7, 201.7)
- moved C11 89.4 mm to (114.7, 163.6)
- moved C15 89.4 mm to (155.7, 185.9)
- moved C16 89.4 mm to (124.2, 201.7)
- moved C17 89.4 mm to (228.5, 163.6)
- moved C18 89.4 mm to (152.7, 163.6)
- moved C19 89.4 mm to (209.6, 163.6)
- moved C21 89.4 mm to (117.8, 185.9)
- moved C24 89.4 mm to (333.4, 125.5)
- moved C25 89.4 mm to (164.3, 201.7)
- moved C27 89.4 mm to (67.7, 185.9)
- moved C28 89.4 mm to (45.7, 201.7)
- moved C29 89.4 mm to (267.1, 163.6)
- moved C3 89.4 mm to (133.0, 163.6)
- moved C31 89.4 mm to (174.9, 185.9)
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Routing:
- net VDD_BAT: track 45.3 -> 49.7 mm
- net LED_POWER: track 48.7 -> 50.8 mm, vias 10 -> 12

Commit message: changed some value fields
Parts:
- C73, C74: value 22µF -> 22uF
- D10, D11, D12, D13, D14, D15, D16, D17, D18, D19, D2, D20, D21, D22, D23, D24, D25, D26, D27, D28, D29, D3, D30, D31, D32, D33, D34, D35, D36, D37, D38, D39, D4, D40, D41, D42, D43, D44, D45, D46, D47, D48, D49, D5, D50, D51, D52, D53, D54, D55, D56, D57, D58, D59, D6, D60, D61, D62, D63, D64, D65, D66, D67, D68, D69, D7, D8, D9: value D_Small -> Switching Diode
- L1: value 22µH -> 22uH
- SW1: value SW_Push -> EVQPUJ02K / EVQPUA02K
Other:
- board text added: "JLCJLCJLCJLC"

Commit message: add lls, switch and spare gpio connector
Parts:
- added J71: Conn_01x04, Connector_PinHeader_2.54mm:PinHeader_1x04_P2.54mm_Horizontal, F.Cu at (360.2, 177.7)
- added R11: 100k, Resistor_SMD:R_0805_2012Metric, F.Cu at (354.1, 156.5)
- added R12: 0R, Resistor_SMD:R_0805_2012Metric, F.Cu at (356.1, 156.5)
- added SW2: SW_SPDT, custom_footprints:SW_SPDT_CK-JS102011SAQN, B.Cu at (365.9, 181.5)
- added U4: SN74LVC1T45DBV, Package_TO_SOT_SMD:SOT-23-6, F.Cu at (351.2, 156.3)
- C1, C2, C74, C75, C76, C77, C78, D1, D10, D12, D13, D14, D140, D141, D15, D17, D18, D19, D2, D20, D21, D22, D23, D24, D25, D27, D28, D29, D3, D30, D31, D32, D33, D34, D35, D36, D37, D38, D39, D40, D41, D42, D43, D44, D45, D46, D47, D48, D49, D50, D51, D52, D53, D54, D55, D56, D57, D58, D60, D61, D63, D64, D65, D66, D67, D68, D7, D8, FB3, Q1, R1, R5, R6, R8: moved to B.Cu
- moved FB3 22.9 mm to (329.2, 123.7), turned to 270 degrees
- moved C76 21.4 mm to (326.8, 127.0)
- moved R4 20.4 mm to (322.6, 123.6)
- moved R3 20.4 mm to (320.7, 123.6)
- moved C1 20.0 mm to (326.8, 125.0)
- moved C78 18.4 mm to (327.0, 116.4)
- moved C77 18.4 mm to (327.0, 118.3)
- moved D1 17.2 mm to (326.6, 122.3)
- moved R1 15.2 mm to (324.2, 117.1)
- moved R2 11.6 mm to (318.8, 114.3)
- moved FB1 11.2 mm to (322.3, 116.4)
- moved FB2 11.2 mm to (321.0, 116.4)
- moved R8 9.04 mm to (326.8, 180.8), turned to 180 degrees
- moved C75 7.64 mm to (318.7, 180.8), turned to 180 degrees
- moved C73 6.73 mm to (316.5, 168.4), turned to 90 degrees
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Connections:
- D13 pad 1: COLUMN_2 -> COLUMN_0
- D18 pad 1: COLUMN_3 -> COLUMN_1
- D23 pad 1: COLUMN_4 -> COLUMN_2
- D24 pad 1: COLUMN_4 -> COLUMN_0
- D28 pad 1: COLUMN_5 -> COLUMN_3
- D29 pad 1: COLUMN_5 -> COLUMN_1
- D31 pad 1: COLUMN_5 -> COLUMN_0
- D32 pad 1: COLUMN_6 -> Net-(D32-Pad1)
- D33 pad 1: COLUMN_6 -> COLUMN_4
- D34 pad 1: COLUMN_6 -> COLUMN_2
- D35 pad 1: COLUMN_6 -> Net-(D32-Pad1)
- D36 pad 1: COLUMN_6 -> COLUMN_1
- D38 pad 1: COLUMN_7 -> COLUMN_5
- D39 pad 1: COLUMN_7 -> COLUMN_3
- D41 pad 1: COLUMN_7 -> COLUMN_2
- D43 pad 1: COLUMN_8 -> Net-(D32-Pad1)
- D44 pad 1: COLUMN_8 -> COLUMN_4
- D46 pad 1: COLUMN_8 -> COLUMN_3
- D47 pad 1: COLUMN_9 -> COLUMN_2
- D48 pad 1: COLUMN_9 -> COLUMN_7
- D49 pad 1: COLUMN_9 -> COLUMN_5
- D50 pad 1: COLUMN_9 -> COLUMN_5
- D51 pad 1: COLUMN_9 -> COLUMN_4
- D52 pad 1: COLUMN_10 -> COLUMN_3
- D53 pad 1: COLUMN_10 -> COLUMN_8
- D54 pad 1: COLUMN_10 -> Net-(D32-Pad1)
- D55 pad 1: COLUMN_10 -> Net-(D32-Pad1)
- D56 pad 1: COLUMN_11 -> COLUMN_4
- D57 pad 1: COLUMN_11 -> COLUMN_4
- D58 pad 1: COLUMN_11 -> COLUMN_7
- D59 pad 1: COLUMN_11 -> COLUMN_7
- D60 pad 1: COLUMN_12 -> COLUMN_5
- D61 pad 1: COLUMN_12 -> COLUMN_5
- D62 pad 1: COLUMN_12 -> COLUMN_8
- D63 pad 1: COLUMN_12 -> COLUMN_8
- D64 pad 1: COLUMN_13 -> Net-(D32-Pad1)
- D65 pad 1: COLUMN_13 -> Net-(D32-Pad1)
- D66 pad 1: COLUMN_14 -> COLUMN_7
- D67 pad 1: COLUMN_14 -> COLUMN_7
- D68 pad 1: COLUMN_15 -> COLUMN_8
- D69 pad 1: COLUMN_15 -> COLUMN_8
- J1 pad 1: VDD_BAT -> Net-(J1-Pad1)
- J10 pad 1: ROW_3 -> ROW_5
- J11 pad 1: ROW_4 -> ROW_6
- J13 pad 1: ROW_1 -> ROW_2
- J14 pad 1: ROW_2 -> ROW_3
- J15 pad 1: ROW_3 -> ROW_5
- J16 pad 1: ROW_4 -> ROW_6
- J18 pad 1: ROW_1 -> ROW_2
- J19 pad 1: ROW_2 -> ROW_3
- J20 pad 1: ROW_3 -> ROW_5
- J21 pad 1: ROW_4 -> ROW_6
- J23 pad 1: ROW_1 -> ROW_2
- J24 pad 1: ROW_2 -> ROW_4
- J25 pad 1: ROW_3 -> ROW_5
- J26 pad 1: ROW_4 -> ROW_6
- J28 pad 1: ROW_1 -> ROW_2
- J29 pad 1: ROW_2 -> ROW_4
- J30 pad 1: ROW_3 -> ROW_5
- J31 pad 1: ROW_4 -> ROW_7
- J33 pad 1: ROW_1 -> ROW_2
- J34 pad 1: ROW_2 -> ROW_4
- J35 pad 1: ROW_3 -> ROW_5
- J36 pad 1: ROW_4 -> ROW_7
- J38 pad 1: ROW_1 -> ROW_2
- J39 pad 1: ROW_2 -> ROW_4
- J4 pad 1: ROW_2 -> ROW_3
- J40 pad 1: ROW_3 -> ROW_5
- J41 pad 1: ROW_4 -> ROW_7
- J43 pad 1: ROW_1 -> ROW_2
- J44 pad 1: ROW_2 -> ROW_4
- J45 pad 1: ROW_3 -> ROW_5
- J46 pad 1: ROW_4 -> ROW_7
- J47 pad 1: ROW_3 -> ROW_6
- J48 pad 1: ROW_4 -> ROW_7
- J49 pad 1: ROW_0 -> ROW_1
- J5 pad 1: ROW_3 -> ROW_5
- J50 pad 1: ROW_1 -> ROW_2
- J51 pad 1: ROW_2 -> ROW_4
- J52 pad 1: ROW_0 -> ROW_1
- J53 pad 1: ROW_1 -> ROW_2
- J54 pad 1: ROW_2 -> ROW_4
- J55 pad 1: ROW_3 -> ROW_6
- J56 pad 1: ROW_0 -> ROW_1
- J57 pad 1: ROW_1 -> ROW_3
- J58 pad 1: ROW_2 -> ROW_4
- J59 pad 1: ROW_3 -> ROW_6
- J6 pad 1: ROW_4 -> ROW_6
- J60 pad 1: ROW_0 -> ROW_1
- J61 pad 1: ROW_1 -> ROW_3
- J62 pad 1: ROW_2 -> ROW_4
- J63 pad 1: ROW_3 -> ROW_6
- J64 pad 1: ROW_0 -> ROW_1
- J65 pad 1: ROW_1 -> ROW_3
- J66 pad 1: ROW_0 -> ROW_1
- J67 pad 1: ROW_1 -> ROW_3
- J68 pad 1: ROW_0 -> ROW_1
- J69 pad 1: ROW_1 -> ROW_3
- J9 pad 1: ROW_2 -> ROW_3
- U2 pad 13: COLUMN_5 -> ROW_3
- U2 pad 15: COLUMN_4 -> ROW_4
- U2 pad 16: COLUMN_3 -> ROW_5
- U2 pad 18: COLUMN_0 -> COLUMN_1
- U2 pad 19: COLUMN_1 -> COLUMN_8
- U2 pad 20: COLUMN_2 -> COLUMN_5
- U2 pad 24: COLUMN_14 -> LLS_INPUT
- U2 pad 26: ROW_2 -> COLUMN_7
- U2 pad 28: COLUMN_6 -> COLUMN_2
- U2 pad 34: COLUMN_13 -> COLUMN_6
- U2 pad 36: COLUMN_12 -> COLUMN_0
- U2 pad 4: ROW_0 -> ROW_1
- U2 pad 40: COLUMN_10 -> COLUMN_3
- U2 pad 42: LED_DATA -> ROW_6
- U2 pad 45: ROW_3 -> ROW_7
- U2 pad 46: COLUMN_11 -> COLUMN_4
- U2 pad 49: COLUMN_7 -> GPIO_3
- U2 pad 51: COLUMN_8 -> GPIO_2
- U2 pad 53: COLUMN_9 -> GPIO_1
- U2 pad 58: ROW_4 -> GPIO_0
- U2 pad 6: ROW_1 -> ROW_2
- U2 pad 8: COLUMN_15 -> ROW_0
Routing:
- net COLUMN_6: track 348.7 -> 0.00 mm, vias 5 -> 0
- net ROW_6: track 0.00 -> 339.4 mm, vias 0 -> 4
- net Net-(D32-Pad1): track 0.00 -> 324.0 mm, vias 0 -> 9
- net ROW_5: track 0.00 -> 322.4 mm, vias 0 -> 2
- net COLUMN_3: track 344.5 -> 592.4 mm, vias 5 -> 11
- net COLUMN_9: track 207.5 -> 0.00 mm, vias 3 -> 0
- net COLUMN_2: track 349.0 -> 511.1 mm, vias 4 -> 16
- net COLUMN_10: track 161.8 -> 0.00 mm, vias 3 -> 0
- net COLUMN_11: track 148.9 -> 0.00 mm, vias 2 -> 0
- net ROW_4: track 360.5 -> 231.0 mm, vias 7 -> 2
- net ROW_7: track 0.00 -> 129.0 mm
- net COLUMN_8: track 220.8 -> 336.4 mm, vias 3 -> 17
- net COLUMN_1: track 376.6 -> 472.7 mm, vias 5 -> 18
- net COLUMN_12: track 94.9 -> 0.00 mm, vias 4 -> 0
- net COLUMN_0: track 382.7 -> 466.2 mm, vias 6 -> 12
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Other:
- board text added: "Keyboard_68 Rev.: 2.1 (c) crohloff"
- board text removed: "Keyboard_68 Rev.: 2.0 (c) crohloff"

Commit message: change usb c connector, fix column 6
Parts:
- removed U1: USB_C, USB_C_Receptacle_Amphenol_12401610E4-2A:USB_C_Receptacle_Amphenol_12401610E4-2A
- added J72: USB_C_Receptacle_USB2.0, custom_footprints:USB_C_China, B.Cu at (323.2, 104.0)
Connections:
- D32 pad 1: Net-(D32-Pad1) -> COLUMN_6
- D35 pad 1: Net-(D32-Pad1) -> COLUMN_6
- D43 pad 1: Net-(D32-Pad1) -> COLUMN_6
- D54 pad 1: Net-(D32-Pad1) -> COLUMN_6
- D55 pad 1: Net-(D32-Pad1) -> COLUMN_6
- D64 pad 1: Net-(D32-Pad1) -> COLUMN_6
- D65 pad 1: Net-(D32-Pad1) -> COLUMN_6
Routing:
- net COLUMN_6: track 0.00 -> 362.2 mm, vias 0 -> 11
- net Net-(D32-Pad1): track 324.0 -> 0.00 mm, vias 9 -> 0
- net Net-(D1-Pad2): track 17.0 -> 24.4 mm, vias 1 -> 3
- net Net-(C1-Pad1): track 29.1 -> 32.6 mm
- net Net-(J72-PadA5): track 6.31 -> 9.06 mm
- net Net-(FB2-Pad2): track 29.2 -> 27.2 mm
- net Net-(D1-Pad3): track 33.6 -> 31.7 mm, vias 4 -> 3
- net Net-(J72-PadB5): track 12.6 -> 11.0 mm
- net Net-(FB1-Pad2): track 19.6 -> 18.0 mm, vias 0 -> 2
