File: Leds.sch (KiCad schematic (older format))
At the start: 140 parts

Commit message: switched to smaller module
Parts:
- D70, D71: footprint LED_SMD:LED_WS2812B_PLCC4_5.0x5.0mm_P3.2mm -> ws2812_inPCB:ws2812_inPCB
Changed lines of the file:
@@
 F 0 "D71" H 4550 1650 50  0000 L CNN
 F 1 "WS2812B" H 4800 1650 50  0000 L CNN
-F 2 "LED_SMD:LED_WS2812B_PLCC4_5.0x5.0mm_P3.2mm" H 4800 1100 50  0001 L TNN
+F 2 "ws2812_inPCB:ws2812_inPCB" H 4800 1100 50  0001 L TNN
 F 3 "https://cdn-shop.adafruit.com/datasheets/WS2812B.pdf" H 4850 1025 50  0001 L TNN
 F 4 "C114585" H 4750 1400 50  0001 C CNN "LCSC"
@@
 F 0 "D70" H 3850 1650 50  0000 L CNN
 F 1 "WS2812B" H 4100 1650 50  0000 L CNN
-F 2 "LED_SMD:LED_WS2812B_PLCC4_5.0x5.0mm_P3.2mm" H 4100 1100 50  0001 L TNN
+F 2 "ws2812_inPCB:ws2812_inPCB" H 4100 1100 50  0001 L TNN
 F 3 "https://cdn-shop.adafruit.com/datasheets/WS2812B.pdf" H 4150 1025 50  0001 L TNN
 F 4 "C114585" H 4050 1400 50  0001 C CNN "LCSC"
